File: keyboard.kicad_pcb (KiCad board)
At the start: 2 copper layers, 549.4 x 162.1 mm, 268 parts

Commit message: Revision 1
Parts:
- K_114, K_115, K_126, K_128: footprint MX_Alps_Hybrid:MX-1.25U-NoLED -> MX_Alps_Hybrid:MX-1U-NoLED
- K_117, K_118, K_124, K_127: footprint MX_Alps_Hybrid:MX-1U-NoLED -> MX_Alps_Hybrid:MX-1.25U-NoLED
- moved K_126 120.4 mm to (148.5, 91.8)
- moved D_126 118.1 mm to (157.0, 92.3)
- moved D_120 113.2 mm to (162.0, 73.9)
- moved D_119 113.2 mm to (143.6, 69.0)
- moved K_119 113.2 mm to (135.1, 68.5)
- moved K_120 113.2 mm to (153.5, 73.4)
- moved K_127 98.9 mm to (21.8, 77.0)
- moved D_127 96.6 mm to (32.7, 77.5)
- moved K_128 96.6 mm to (116.0, 102.9)
- moved D_128 94.3 mm to (124.5, 103.4)
- moved D_115 53.4 mm to (47.0, 43.1)
- moved K_117 51.3 mm to (86.8, 55.0)
- moved K_115 51.1 mm to (38.4, 42.6)
- moved D_117 49.0 mm to (97.7, 55.5)
- moved D_116 48.8 mm to (74.7, 49.3)
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Connections:
- D_115 pad 1: row3 -> row2
- D_116 pad 1: row3 -> row2
- D_119 pad 1: row2 -> row3
- D_120 pad 1: row2 -> row3
- D_123 pad 1: row4 -> row3
- D_126 pad 1: row3 -> row4
- D_127 pad 1: row5 -> row4
- D_128 pad 1: row4 -> row5
- K_107 pad 1: col7 -> col6
- K_114 pad 1: col3 -> col0
- K_115 pad 1: col4 -> col1
- K_116 pad 1: col5 -> col3
- K_117 pad 1: col7 -> col4
- K_118 pad 1: col7 -> col5
- K_119 pad 1: col1 -> col6
- K_120 pad 1: col2 -> col7
- K_121 pad 1: col3 -> col1
- K_122 pad 1: col4 -> col2
- K_123 pad 1: col5 -> col4
- K_124 pad 1: col6 -> col5
- K_125 pad 1: col7 -> col6
- K_126 pad 1: col1 -> col7
- K_127 pad 1: col6 -> col0
- K_128 pad 1: col0 -> col5
- K_130 pad 1: col8 -> col7
- K_71 pad 1: col23 -> col22
- K_93 pad 1: col11 -> col10
- K_95 pad 1: col16 -> col15
- K_97 pad 1: col21 -> col20
Other:
- board size 549.4 x 162.1 mm -> 548.1 x 162.1 mm
